File: hw/airplane-keychain.kicad_sch (KiCad schematic)
At the start: 19 parts, among them IC1 ATTINY85-P, J1 CONN_01X03_MALE, SW1 SW_PUSH, SW2 SPST

Commit message: KiCad update
Parts:
- removed IC1: ATTINY85-P, Housings_DIP:DIP-8_W7.62mm, symbol airplane-keychain-rescue:ATTINY85-P
- added U1: ATtiny85-20P, Package_DIP:DIP-8_W7.62mm, symbol MCU_Microchip_ATtiny:ATtiny85-20P
Connections:
- net GND: now also U1.4 (GND)
- net at D5.2 (A), D6.2 (A): now also U1.3 (XTAL2/PB4)
- net at R6.2: now also U1.1 (~{RESET}/PB5)
- net at R4.1: now also U1.2 (XTAL1/PB3)
- net at R1.1: now also U1.5 (AREF/PB0)
- net at R2.1: now also U1.6 (PB1)
- net at R3.1: now also U1.7 (PB2)
- net at R6.1, SW2.1: now also U1.8 (VCC)
Other:
- company: (none) -> Make to Innovate

Commit message: Added Gerbers
Parts:
- BT1, BT2: footprint Battery_Holders:Keystone_1058_1x2032-CoinCell -> Battery:BatteryHolder_Keystone_1058_1x2032
- D1: footprint LEDs:LED_D5.0mm -> LED_THT:LED_D5.0mm_FlatTop
- D2, D5, D6: footprint LEDs:LED_1206 -> LED_SMD:LED_1206_3216Metric_Pad1.42x1.75mm_HandSolder
- D3, D4: footprint LEDs:LED_D3.0mm_Horizontal_O1.27mm_Z2.0mm -> LED_THT:LED_D3.0mm_Horizontal_O1.27mm_Z2.0mm_Clear
- D7: footprint LEDs:LED_D5.0mm_Horizontal_O1.27mm_Z3.0mm -> LED_THT:LED_D5.0mm_Horizontal_O1.27mm_Z3.0mm_Clear
- J1: footprint Pin_Headers:Pin_Header_Straight_1x03_Pitch2.54mm -> Connector_PinHeader_2.54mm:PinHeader_1x03_P2.54mm_Vertical
- R1, R2, R3, R4, R5, R6: footprint Resistors_THT:R_Axial_DIN0309_L9.0mm_D3.2mm_P12.70mm_Horizontal -> Resistor_THT:R_Axial_DIN0309_L9.0mm_D3.2mm_P12.70mm_Horizontal
- SW1: footprint Buttons_Switches_THT:SW_PUSH_6mm -> Button_Switch_THT:SW_PUSH_6mm_H5mm
- SW2: footprint Buttons_Switches_THT:SW_Micro_SPST -> Button_Switch_THT:SW_DIP_SPSTx01_Slide_6.7x4.1mm_W7.62mm_P2.54mm_LowProfile
Changed lines of the file:
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@@
       (effects (font (size 1.27 1.27)))
     )
-    (property "Footprint" "LEDs:LED_D5.0mm" (at 55.88 50.8 0)
+    (property "Footprint" "LED_THT:LED_D5.0mm_FlatTop" (at 55.88 50.8 0)
       (effects (font (size 1.27 1.27)) hide)
     )
@@
       (effects (font (size 1.27 1.27)))
     )
-    (property "Footprint" "LEDs:LED_1206" (at 55.88 59.69 0)
+    (property "Footprint" "LED_SMD:LED_1206_3216Metric_Pad1.42x1.75mm_HandSolder" (at 55.88 59.69 0)
       (effects (font (size 1.27 1.27)) hide)
     )
@@
       (effects (font (size 1.27 1.27)))
     )
-    (property "Footprint" "LEDs:LED_D3.0mm_Horizontal_O1.27mm_Z2.0mm" (at 55.88 71.12 0)
+    (property "Footprint" "LED_THT:LED_D3.0mm_Horizontal_O1.27mm_Z2.0mm_Clear" (at 55.88 71.12 0)
       (effects (font (size 1.27 1.27)) hide)
     )
@@
       (effects (font (size 1.27 1.27)))
     )
-    (property "Footprint" "LEDs:LED_D3.0mm_Horizontal_O1.27mm_Z2.0mm" (at 55.88 80.01 0)
+    (property "Footprint" "LED_THT:LED_D3.0mm_Horizontal_O1.27mm_Z2.0mm_Clear" (at 55.88 80.01 0)
       (effects (font (size 1.27 1.27)) hide)
     )
@@
       (effects (font (size 1.27 1.27)))
     )
-    (property "Footprint" "LEDs:LED_1206" (at 55.88 93.98 0)
+    (property "Footprint" "LED_SMD:LED_1206_3216Metric_Pad1.42x1.75mm_HandSolder" (at 55.88 93.98 0)
       (effects (font (size 1.27 1.27)) hide)
     )
@@
       (effects (font (size 1.27 1.27)))
     )
-    (property "Footprint" "LEDs:LED_1206" (at 55.88 102.87 0)
+    (property "Footprint" "LED_SMD:LED_1206_3216Metric_Pad1.42x1.75mm_HandSolder" (at 55.88 102.87 0)
       (effects (font (size 1.27 1.27)) hide)
     )
@@
       (effects (font (size 1.27 1.27)))
     )
-    (property "Footprint" "LEDs:LED_D5.0mm_Horizontal_O1.27mm_Z3.0mm" (at 55.88 116.84 0)
+    (property "Footprint" "LED_THT:LED_D5.0mm_Horizontal_O1.27mm_Z3.0mm_Clear" (at 55.88 116.84 0)
       (effects (font (size 1.27 1.27)) hide)
     )
@@
       (effects (font (size 1.27 1.27)))
     )
-    (property "Footprint" "Buttons_Switches_THT:SW_PUSH_6mm" (at 106.68 116.84 0)
+    (property "Footprint" "Button_Switch_THT:SW_PUSH_6mm_H5mm" (at 106.68 116.84 0)
       (effects (font (size 1.27 1.27)) hide)
     )
@@
       (effects (font (size 1.27 1.27)))
     )
-    (property "Footprint" "Buttons_Switches_THT:SW_Micro_SPST" (at 220.98 87.63 0)
+    (property "Footprint" "Button_Switch_THT:SW_DIP_SPSTx01_Slide_6.7x4.1mm_W7.62mm_P2.54mm_LowProfile" (at 220.98 87.63 0)
       (effects (font (size 1.27 1.27)) hide)
     )
@@
       (effects (font (size 1.27 1.27)))
     )
-    (property "Footprint" "Resistors_THT:R_Axial_DIN0309_L9.0mm_D3.2mm_P12.70mm_Horizontal" (at 74.93 49.022 90)
+    (property "Footprint" "Resistor_THT:R_Axial_DIN0309_L9.0mm_D3.2mm_P12.70mm_Horizontal" (at 74.93 49.022 90)
       (effects (font (size 1.27 1.27)) hide)
     )
@@
       (effects (font (size 1.27 1.27)))
     )
-    (property "Footprint" "Resistors_THT:R_Axial_DIN0309_L9.0mm_D3.2mm_P12.70mm_Horizontal" (at 74.93 57.912 90)
+    (property "Footprint" "Resistor_THT:R_Axial_DIN0309_L9.0mm_D3.2mm_P12.70mm_Horizontal" (at 74.93 57.912 90)
       (effects (font (size 1.27 1.27)) hide)
     )
@@
       (effects (font (size 1.27 1.27)))
     )
-    (property "Footprint" "Resistors_THT:R_Axial_DIN0309_L9.0mm_D3.2mm_P12.70mm_Horizontal" (at 74.93 69.342 90)
+    (property "Footprint" "Resistor_THT:R_Axial_DIN0309_L9.0mm_D3.2mm_P12.70mm_Horizontal" (at 74.93 69.342 90)
       (effects (font (size 1.27 1.27)) hide)
     )
@@
       (effects (font (size 1.27 1.27)))
     )
-    (property "Footprint" "Resistors_THT:R_Axial_DIN0309_L9.0mm_D3.2mm_P12.70mm_Horizontal" (at 74.93 78.232 90)
+    (property "Footprint" "Resistor_THT:R_Axial_DIN0309_L9.0mm_D3.2mm_P12.70mm_Horizontal" (at 74.93 78.232 90)
       (effects (font (size 1.27 1.27)) hide)
     )
@@
       (effects (font (size 1.27 1.27)))
     )
-    (property "Footprint" "Resistors_THT:R_Axial_DIN0309_L9.0mm_D3.2mm_P12.70mm_Horizontal" (at 74.93 115.062 90)
+    (property "Footprint" "Resistor_THT:R_Axial_DIN0309_L9.0mm_D3.2mm_P12.70mm_Horizontal" (at 74.93 115.062 90)
       (effects (font (size 1.27 1.27)) hide)
     )
@@
       (effects (font (size 1.27 1.27)) (justify left))
     )
-    (property "Footprint" "Battery_Holders:Keystone_1058_1x2032-CoinCell" (at 234.95 117.856 90)
+    (property "Footprint" "Battery:BatteryHolder_Keystone_1058_1x2032" (at 234.95 117.856 90)
       (effects (font (size 1.27 1.27)) hide)
     )
@@
       (effects (font (size 1.27 1.27)) (justify left))
     )
-    (property "Footprint" "Battery_Holders:Keystone_1058_1x2032-CoinCell" (at 220.98 117.856 90)
+    (property "Footprint" "Battery:BatteryHolder_Keystone_1058_1x2032" (at 220.98 117.856 90)
       (effects (font (size 1.27 1.27)) hide)
     )
@@
       (effects (font (size 1.27 1.27)))
     )
-    (property "Footprint" "Pin_Headers:Pin_Header_Straight_1x03_Pitch2.54mm" (at 48.26 26.67 0)
+    (property "Footprint" "Connector_PinHeader_2.54mm:PinHeader_1x03_P2.54mm_Vertical" (at 48.26 26.67 0)
       (effects (font (size 1.27 1.27)) hide)
     )
@@
       (effects (font (size 1.27 1.27)))
     )
-    (property "Footprint" "Resistors_THT:R_Axial_DIN0309_L9.0mm_D3.2mm_P12.70mm_Horizontal" (at 161.29 99.822 90)
-      (effects (font (size 1.27 1.27)) hide)
-    )
+    (property "Footprint" "Resistor_THT:R_Axial_DIN0309_L9.0mm_D3.2mm_P12.70mm_Horizontal" (at 161.29 99.822 90)
+      (effects (font (size 1.27 1.27)) hide)
+    )

Commit message: updates
Parts:
- removed R6: 10k, Resistor_THT:R_Axial_DIN0309_L9.0mm_D3.2mm_P12.70mm_Horizontal, symbol airplane-keychain-rescue:R
- removed U1: ATtiny85-20P, Package_DIP:DIP-8_W7.62mm, symbol MCU_Microchip_ATtiny:ATtiny85-20P
- added U2: ~, symbol MCU_Module:adafruit_qtpy_SAMD
Connections:
- net GND: now also U2.12 (GND)
- net at D5.2 (A): now also U2.0 (A0); no longer D6.2 (A)
- net at R1.1: now also U2.3 (A3)
- new net: D6.2 (A), U2.1 (A1)
Changed lines of the file:
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@@
   (junction (at 40.64 50.8) (diameter 0) (color 0 0 0 0)
   )
-  (junction (at 207.01 90.17) (diameter 0) (color 0 0 0 0)
-  )
-  (junction (at 118.11 93.98) (diameter 0) (color 0 0 0 0)
-  )
   (junction (at 40.64 93.98) (diameter 0) (color 0 0 0 0)
   )
@@
   (junction (at 220.98 124.46) (diameter 0) (color 0 0 0 0)
   )
-  (wire (pts (xy 139.7 69.85) (xy 139.7 101.6))
-    (stroke (width 0) (type default))
-  )
   (wire (pts (xy 60.96 50.8) (xy 63.5 50.8))
     (stroke (width 0) (type default))
@@
     (stroke (width 0) (type default))
   )
-  (wire (pts (xy 146.05 80.01) (xy 137.16 80.01))
-    (stroke (width 0) (type default))
-  )
   (wire (pts (xy 40.64 59.69) (xy 40.64 71.12))
     (stroke (width 0) (type default))
@@
     (stroke (width 0) (type default))
   )
-  (wire (pts (xy 146.05 72.39) (xy 134.62 72.39))
+  (wire (pts (xy 152.4 102.87) (xy 152.4 59.69))
     (stroke (width 0) (type default))
   )
@@
     (stroke (width 0) (type default))
   )
-  (wire (pts (xy 132.08 77.47) (xy 132.08 71.12))
-    (stroke (width 0) (type default))
-  )
-  (wire (pts (xy 60.96 93.98) (xy 118.11 93.98))
+  (wire (pts (xy 152.4 59.69) (xy 170.18 59.69))
+    (stroke (width 0) (type default))
+  )
+  (wire (pts (xy 60.96 93.98) (xy 156.21 93.98))
     (stroke (width 0) (type default))
   )
@@
     (stroke (width 0) (type default))
   )
-  (wire (pts (xy 137.16 59.69) (xy 137.16 80.01))
+  (wire (pts (xy 156.21 57.15) (xy 170.18 57.15))
     (stroke (width 0) (type default))
   )
@@
     (stroke (width 0) (type default))
   )
-  (wire (pts (xy 114.3 80.01) (xy 114.3 74.93))
-    (stroke (width 0) (type default))
-  )
   (wire (pts (xy 220.98 121.92) (xy 220.98 124.46))
     (stroke (width 0) (type default))
@@
     (stroke (width 0) (type default))
   )
+  (wire (pts (xy 160.02 50.8) (xy 160.02 64.77))
+    (stroke (width 0) (type default))
+  )
   (wire (pts (xy 63.5 36.83) (xy 63.5 50.8))
     (stroke (width 0) (type default))
   )
-  (wire (pts (xy 207.01 90.17) (xy 207.01 101.6))
+  (wire (pts (xy 160.02 64.77) (xy 170.18 64.77))
     (stroke (width 0) (type default))
   )
@@
     (stroke (width 0) (type default))
   )
-  (wire (pts (xy 161.29 90.17) (xy 207.01 90.17))
-    (stroke (width 0) (type default))
-  )
   (wire (pts (xy 234.95 107.95) (xy 234.95 114.3))
     (stroke (width 0) (type default))
@@
     (stroke (width 0) (type default))
   )
-  (wire (pts (xy 118.11 102.87) (xy 60.96 102.87))
-    (stroke (width 0) (type default))
-  )
-  (wire (pts (xy 146.05 77.47) (xy 132.08 77.47))
-    (stroke (width 0) (type default))
-  )
-  (wire (pts (xy 134.62 72.39) (xy 134.62 80.01))
+  (wire (pts (xy 60.96 102.87) (xy 152.4 102.87))
     (stroke (width 0) (type default))
   )
@@
     (stroke (width 0) (type default))
   )
-  (wire (pts (xy 146.05 82.55) (xy 142.24 82.55))
-    (stroke (width 0) (type default))
-  )
-  (wire (pts (xy 118.11 80.01) (xy 118.11 93.98))
-    (stroke (width 0) (type default))
-  )
   (wire (pts (xy 50.8 93.98) (xy 40.64 93.98))
     (stroke (width 0) (type default))
   )
-  (wire (pts (xy 146.05 69.85) (xy 139.7 69.85))
-    (stroke (width 0) (type default))
-  )
   (wire (pts (xy 78.74 59.69) (xy 137.16 59.69))
     (stroke (width 0) (type default))
@@
     (stroke (width 0) (type default))
   )
-  (wire (pts (xy 207.01 69.85) (xy 207.01 90.17))
-    (stroke (width 0) (type default))
-  )
   (wire (pts (xy 50.8 116.84) (xy 40.64 116.84))
     (stroke (width 0) (type default))
@@
     (stroke (width 0) (type default))
   )
-  (wire (pts (xy 139.7 101.6) (xy 157.48 101.6))
-    (stroke (width 0) (type default))
-  )
-  (wire (pts (xy 78.74 50.8) (xy 142.24 50.8))
+  (wire (pts (xy 187.96 59.69) (xy 196.85 59.69))
+    (stroke (width 0) (type default))
+  )
+  (wire (pts (xy 156.21 93.98) (xy 156.21 57.15))
+    (stroke (width 0) (type default))
+  )
+  (wire (pts (xy 78.74 50.8) (xy 160.02 50.8))
     (stroke (width 0) (type default))
   )
@@
     (stroke (width 0) (type default))
   )
-  (wire (pts (xy 161.29 54.61) (xy 161.29 59.69))
-    (stroke (width 0) (type default))
-  )
   (wire (pts (xy 50.8 80.01) (xy 40.64 80.01))
     (stroke (width 0) (type default))
@@
     (stroke (width 0) (type default))
   )
-  (wire (pts (xy 114.3 74.93) (xy 146.05 74.93))
-    (stroke (width 0) (type default))
-  )
   (wire (pts (xy 220.98 69.85) (xy 220.98 74.93))
     (stroke (width 0) (type default))
@@
     (stroke (width 0) (type default))
   )
-  (wire (pts (xy 165.1 101.6) (xy 207.01 101.6))
-    (stroke (width 0) (type default))
-  )
-  (wire (pts (xy 118.11 80.01) (xy 134.62 80.01))
-    (stroke (width 0) (type default))
-  )
   (wire (pts (xy 63.5 50.8) (xy 71.12 50.8))
     (stroke (width 0) (type default))
   )
-  (wire (pts (xy 207.01 69.85) (xy 220.98 69.85))
-    (stroke (width 0) (type default))
-  )
   (wire (pts (xy 234.95 121.92) (xy 234.95 124.46))
     (stroke (width 0) (type default))
@@
     (stroke (width 0) (type default))
   )
-  (wire (pts (xy 142.24 50.8) (xy 142.24 82.55))
-    (stroke (width 0) (type default))
-  )
   (wire (pts (xy 40.64 102.87) (xy 40.64 116.84))
-    (stroke (width 0) (type default))
-  )
-  (wire (pts (xy 118.11 93.98) (xy 118.11 102.87))
     (stroke (width 0) (type default))
   )
@@
     )
   )
-  (symbol (lib_id "airplane-keychain-rescue:GND") (at 161.29 54.61 180) (unit 1)
-    (in_bom yes) (on_board yes) (dnp no)
-    (property "Reference" "#PWR01" (at 161.29 48.26 0)
-      (effects (font (size 1.27 1.27)) hide)
-    )
-    (property "Value" "GND" (at 161.29 50.8 0)
-      (effects (font (size 1.27 1.27)))
-    )
-    (property "Footprint" "" (at 161.29 54.61 0)
-      (effects (font (size 1.27 1.27)))
-    )
-    (property "Datasheet" "" (at 161.29 54.61 0)
+  (symbol (lib_id "airplane-keychain-rescue:GND") (at 196.85 59.69 90) (unit 1)
+    (in_bom yes) (on_board yes) (dnp no)
+    (property "Reference" "#PWR01" (at 203.2 59.69 0)
+      (effects (font (size 1.27 1.27)) hide)
+    )
+    (property "Value" "GND" (at 200.66 59.69 0)
+      (effects (font (size 1.27 1.27)))
+    )
+    (property "Footprint" "" (at 196.85 59.69 0)
+      (effects (font (size 1.27 1.27)))
+    )
+    (property "Datasheet" "" (at 196.85 59.69 0)
       (effects (font (size 1.27 1.27)))
     )
@@
     )
   )
-  (symbol (lib_id "airplane-keychain-rescue:R") (at 161.29 101.6 270) (unit 1)
-    (in_bom yes) (on_board yes) (dnp no)
-    (property "Reference" "R6" (at 161.29 103.632 90)
-      (effects (font (size 1.27 1.27)))
-    )
-    (property "Value" "10k" (at 161.29 101.6 90)
-      (effects (font (size 1.27 1.27)))
-    )
-    (property "Footprint" "Resistor_THT:R_Axial_DIN0309_L9.0mm_D3.2mm_P12.70mm_Horizontal" (at 161.29 99.822 90)
-      (effects (font (size 1.27 1.27)) hide)
-    )
-    (property "Datasheet" "" (at 161.29 101.6 0)
-      (effects (font (size 1.27 1.27)) hide)
-    )
-    (pin "1")
-    (pin "2")
-    (instances
-      (project "airplane-keychain"
-        (path "/6cfc2c66-5048-4a9e-b97d-b82fde315677"
-          (reference "R6") (unit 1)
-        )
-      )
-    )
-  )
-  (symbol (lib_id "MCU_Microchip_ATtiny:ATtiny85-20P") (at 161.29 74.93 180) (unit 1)
+  (symbol (lib_id "MCU_Module:adafruit_qtpy_SAMD") (at 179.07 63.5 0) (unit 1)
     (in_bom yes) (on_board yes) (dnp no) (fields_autoplaced)
-    (property "Reference" "U1" (at 175.26 74.295 0)
-      (effects (font (size 1.27 1.27)) (justify right))
-    )
-    (property "Value" "ATtiny85-20P" (at 175.26 76.835 0)
-      (effects (font (size 1.27 1.27)) (justify right))
-    )
-    (property "Footprint" "Package_DIP:DIP-8_W7.62mm" (at 161.29 74.93 0)
-      (effects (font (size 1.27 1.27) italic) hide)
-    )
-    (property "Datasheet" "http://ww1.microchip.com/downloads/en/DeviceDoc/atmel-2586-avr-8-bit-microcontroller-attiny25-attiny45-attiny85_datasheet.pdf" (at 161.29 74.93 0)
-      (effects (font (size 1.27 1.27)) hide)
-    )
-    (pin "1")
+    (property "Reference" "U2" (at 179.07 52.07 0)
+      (effects (font (size 1.27 1.27)))
+    )
+    (property "Value" "~" (at 179.07 63.5 0)
+      (effects (font (size 1.27 1.27)))
+    )
+    (property "Footprint" "" (at 179.07 63.5 0)
+      (effects (font (size 1.27 1.27)) hide)
+    )
+    (property "Datasheet" "" (at 179.07 63.5 0)
+      (effects (font (size 1.27 1.27)) hide)
+    )
+    (pin "0")
+    (pin "1")
+    (pin "10")
+    (pin "11")
+    (pin "12")
+    (pin "13")
     (pin "2")
     (pin "3")
@@
     (pin "7")
     (pin "8")
-    (instances
-      (project "airplane-keychain"
-        (path "/6cfc2c66-5048-4a9e-b97d-b82fde315677"
-          (reference "U1") (unit 1)
-        )
-      )
+    (pin "9")
+    (instances
+      (project "airplane-keychain"
+        (path "/6cfc2c66-5048-4a9e-b97d-b82fde315677"
+          (reference "U2") (unit 1)
+        )
+      )
