File: hw/airplane-keychain.kicad_pcb (KiCad board)
At the start: 2 copper layers, 93.7 x 109.7 mm, 26 parts, among them SW1 SW_PUSH, SW2 SPST, U1 ATtiny85-20P

Commit message: Final update
Parts:
- moved D9 48.4 mm to (120.6, 74.8)
- moved R10 36.5 mm to (101.3, 101.3), turned to 90 degrees
- moved SW1 6.97 mm to (101.3, 110.7)
- moved D7 3.66 mm to (156.4, 112.2), turned to -90 degrees
- moved D5 0.12 mm to (115.1, 78.1)
Routing:
- net Net-(D8-A): track 0.00 -> 40.4 mm
- net Net-(D9-A): track 0.00 -> 27.6 mm
- net Net-(R10-Pad1): track 62.8 -> 79.6 mm
- net Net-(D7-A): track 0.00 -> 8.19 mm
- net Net-(BT1-+): track 92.2 -> 94.8 mm
Other:
- board text added: "PCB3D_BR_ISGCLOGO"
- board text added: "PCB3D_TL_ISGCLOGO"
Changed lines of the file:
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@@
   )
   (footprint "LED_THT:LED_D3.0mm" (layer "F.Cu")
-    (at 115.2 78.2 180)
+    (at 115.14 78.1 180)
     (descr "LED, diameter 3.0mm, 2 pins")
     (tags "LED diameter 3.0mm 2 pins")
@@
     (property "Sheetname" "")
     (attr through_hole)
-    (fp_text reference "R1" (at 6.35 -2.72 150) (layer "F.SilkS")
+    (fp_text reference "R1" (at 8.608142 -2.487307 150) (layer "F.SilkS")
         (effects (font (size 1 1) (thickness 0.15)))
     )
@@
   )
   (footprint "Button_Switch_THT:SW_PUSH_6mm" (layer "F.Cu")
-    (at 100.3 103.8 180)
+    (at 101.3 110.7 180)
     (descr "https://www.omron.com/ecb/products/pdf/en-b3f.pdf")
     (tags "tact sw push 6mm")
@@
   )
   (footprint "LED_THT:LED_D3.0mm" (layer "F.Cu")
-    (at 157 115.84 90)
+    (at 156.4 112.225 -90)
     (descr "LED, diameter 3.0mm, 2 pins")
     (tags "LED diameter 3.0mm 2 pins")
@@
     (fp_circle (center 1.27 0) (end 2.77 0)
       (stroke (width 0.1) (type solid)) (fill none) (layer "F.Fab"))
-    (pad "1" thru_hole rect (at 0 0 90) (size 1.8 1.8) (drill 0.9) (layers "*.Cu" "*.Mask")
+    (pad "1" thru_hole rect (at 0 0 270) (size 1.8 1.8) (drill 0.9) (layers "*.Cu" "*.Mask")
       (net 1 "GND") (pinfunction "K") (pintype "passive"))
-    (pad "2" thru_hole circle (at 2.54 0 90) (size 1.8 1.8) (drill 0.9) (layers "*.Cu" "*.Mask")
+    (pad "2" thru_hole circle (at 2.54 0 270) (size 1.8 1.8) (drill 0.9) (layers "*.Cu" "*.Mask")
       (net 9 "Net-(D7-A)") (pinfunction "A") (pintype "passive"))
     (model "${KICAD6_3DMODEL_DIR}/LED_THT.3dshapes/LED_D3.0mm.wrl"
@@
   )
   (footprint "Resistor_THT:R_Axial_DIN0309_L9.0mm_D3.2mm_P12.70mm_Horizontal" (layer "F.Cu")
-    (at 129.54 124.46)
+    (at 101.3 101.3 90)
     (descr "Resistor, Axial_DIN0309 series, Axial, Horizontal, pin pitch=12.7mm, 0.5W = 1/2W, length*diameter=9*3.2mm^2, http://cdn-reichelt.de/documents/datenblatt/B400/1_4W%23YAG.pdf")
     (tags "Resistor Axial_DIN0309 series Axial Horizontal pin pitch 12.7mm 0.5W = 1/2W length 9mm diameter 3.2mm")
@@
     (property "Sheetname" "")
     (attr through_hole)
-    (fp_text reference "R10" (at 6.35 -2.72) (layer "F.SilkS")
+    (fp_text reference "R10" (at 6.35 -2.72 90) (layer "F.SilkS")
         (effects (font (size 1 1) (thickness 0.15)))
     )
-    (fp_text value "100" (at 6.35 2.72) (layer "F.Fab")
+    (fp_text value "100" (at 6.35 2.72 90) (layer "F.Fab")
         (effects (font (size 1 1) (thickness 0.15)))
     )
-    (fp_text user "${REFERENCE}" (at 6.35 0) (layer "F.Fab")
+    (fp_text user "${REFERENCE}" (at 6.35 0 90) (layer "F.Fab")
         (effects (font (size 1 1) (thickness 0.15)))
     )
@@
     (fp_line (start 12.7 0) (end 10.85 0)
       (stroke (width 0.1) (type solid)) (layer "F.Fab"))
-    (pad "1" thru_hole circle (at 0 0) (size 1.6 1.6) (drill 0.8) (layers "*.Cu" "*.Mask")
+    (pad "1" thru_hole circle (at 0 0 90) (size 1.6 1.6) (drill 0.8) (layers "*.Cu" "*.Mask")
       (net 19 "Net-(R10-Pad1)") (pintype "passive"))
-    (pad "2" thru_hole oval (at 12.7 0) (size 1.6 1.6) (drill 0.8) (layers "*.Cu" "*.Mask")
+    (pad "2" thru_hole oval (at 12.7 0 90) (size 1.6 1.6) (drill 0.8) (layers "*.Cu" "*.Mask")
       (net 2 "Net-(D9-A)") (pintype "passive"))
     (model "${KICAD6_3DMODEL_DIR}/Resistor_THT.3dshapes/R_Axial_DIN0309_L9.0mm_D3.2mm_P12.70mm_Horizontal.wrl"
@@
   )
   (footprint "LED_THT:LED_D3.0mm" (layer "F.Cu")
-    (at 162.56 99.06)
+    (at 120.625 74.8)
     (descr "LED, diameter 3.0mm, 2 pins")
     (tags "LED diameter 3.0mm 2 pins")
@@
   (gr_line (start 131 150.9) (end 84.1 123.6)
     (stroke (width 0.15) (type default)) (layer "Edge.Cuts"))
-  (gr_text "ISGC Badge Rev A\nMatthew E. Nelson" (at 135.8 97.6) (layer "B.SilkS")
+  (gr_text "PCB3D_BR_ISGCLOGO" (at 82.4 152.5) (layer "B.Cu")
+    (effects (font (size 1.5 1.5) (thickness 0.3) bold) (justify left bottom mirror))
+  )
+  (gr_text "ISGC Badge Rev A\nMatthew E. Nelson" (at 136.9 98.6) (layer "B.SilkS")
     (effects (font (size 1 1) (thickness 0.15)) (justify left bottom mirror))
   )
-  (segment (start 95.6 89.8) (end 95.6 97.5) (width 0.25) (layer "F.Cu") (net 3))
-  (segment (start 95.6 97.5) (end 93.8 99.3) (width 0.25) (layer "F.Cu") (net 3))
+  (gr_text "PCB3D_TL_ISGCLOGO" (at 181.5 40.2) (layer "F.SilkS")
+    (effects (font (size 1.5 1.5) (thickness 0.3) bold) (justify left bottom mirror))
+  )
+  (segment (start 101.3 88.6) (end 109.365 88.6) (width 0.25) (layer "B.Cu") (net 2))
+  (segment (start 109.365 88.6) (end 123.165 74.8) (width 0.25) (layer "B.Cu") (net 2))
+  (segment (start 94.800001 90.599999) (end 95.6 89.8) (width 0.25) (layer "F.Cu") (net 3))
+  (segment (start 94.8 106.2) (end 94.800001 90.599999) (width 0.25) (layer "F.Cu") (net 3))
   (segment (start 145.1 85.8) (end 145.1 109.9) (width 0.25) (layer "B.Cu") (net 3))
   (segment (start 145.1 109.9) (end 145.5 110.3) (width 0.25) (layer "B.Cu") (net 3))
   (segment (start 145.5 86.2) (end 145.1 85.8) (width 0.25) (layer "B.Cu") (net 3))
-  (segment (start 145.5 110.3) (end 122.8 110.3) (width 0.25) (layer "B.Cu") (net 3))
-  (segment (start 122.8 110.3) (end 111.8 99.3) (width 0.25) (layer "B.Cu") (net 3))
-  (segment (start 100.3 99.3) (end 93.8 99.3) (width 0.25) (layer "B.Cu") (net 3))
-  (segment (start 111.8 99.3) (end 100.3 99.3) (width 0.25) (layer "B.Cu") (net 3))
+  (segment (start 94.8 106.2) (end 101.3 106.2) (width 0.25) (layer "B.Cu") (net 3))
+  (segment (start 141.4 106.2) (end 145.5 110.3) (width 0.25) (layer "B.Cu") (net 3))
+  (segment (start 101.3 106.2) (end 141.4 106.2) (width 0.25) (layer "B.Cu") (net 3))
   (segment (start 145.5 110.3) (end 145.5 109.815) (width 0.25) (layer "B.Cu") (net 3))
   (segment (start 166.4 73.3) (end 169.925 76.825) (width 0.25) (layer "F.Cu") (net 4))
@@
   (segment (start 159.96 107.6) (end 159.96 102.04) (width 0.25) (layer "F.Cu") (net 7))
   (segment (start 159.96 102.04) (end 167 95) (width 0.25) (layer "F.Cu") (net 7))
-  (segment (start 92.425 114.625) (end 92.425 83.105) (width 0.25) (layer "F.Cu") (net 8))
-  (segment (start 97.33 78.2) (end 112.66 78.2) (width 0.25) (layer "F.Cu") (net 8))
+  (segment (start 92.425 83.105) (end 97.43 78.1) (width 0.25) (layer "F.Cu") (net 8))
   (segment (start 95.5 117.7) (end 92.425 114.625) (width 0.25) (layer "F.Cu") (net 8))
-  (segment (start 92.425 83.105) (end 97.33 78.2) (width 0.25) (layer "F.Cu") (net 8))
+  (segment (start 92.425 114.625) (end 92.425 83.105) (width 0.25) (layer "F.Cu") (net 8))
+  (segment (start 97.43 78.1) (end 112.6 78.1) (width 0.25) (layer "F.Cu") (net 8))
+  (segment (start 156.4 114.765) (end 156.4 117.245738) (width 0.25) (layer "F.Cu") (net 9))
+  (segment (start 156.4 117.245738) (end 160.439262 121.285) (width 0.25) (layer "F.Cu") (net 9))
   (segment (start 155.401477 66.95) (end 148.57 66.95) (width 0.25) (layer "F.Cu") (net 10))
   (segment (start 148.57 66.95) (end 148.2 66.58) (width 0.25) (layer "F.Cu") (net 10))
@@
   (segment (start 91.975 115.765991) (end 91.975 82.918604) (width 0.25) (layer "F.Cu") (net 16))
   (segment (start 98.793604 76.1) (end 103.26 76.1) (width 0.25) (layer "F.Cu") (net 16))
+  (segment (start 155.8 109.5) (end 163.5 109.5) (width 0.25) (layer "F.Cu") (net 17))
+  (segment (start 163.5 109.5) (end 168.7 104.3) (width 0.25) (layer "F.Cu") (net 17))
+  (segment (start 144.799262 120.500738) (end 155.8 109.5) (width 0.25) (layer "F.Cu") (net 17))
+  (segment (start 144.799262 130.325) (end 144.799262 120.500738) (width 0.25) (layer "F.Cu") (net 17))
   (segment (start 145.66 89.191477) (end 110.801477 124.05) (width 0.25) (layer "F.Cu") (net 18))
   (segment (start 110.801477 124.05) (end 117.201477 130.45) (width 0.25) (layer "F.Cu") (net 18))
   (segment (start 106.498523 124.05) (end 110.801477 124.05) (width 0.25) (layer "F.Cu") (net 18))
   (segment (start 145.66 74.2) (end 145.66 89.191477) (width 0.25) (layer "F.Cu") (net 18))
-  (segment (start 100.3 103.8) (end 100.3 119.442468) (width 0.25) (layer "F.Cu") (net 19))
-  (segment (start 128.700739 131.575) (end 133.800739 136.675) (width 0.25) (layer "F.Cu") (net 19))
-  (segment (start 100.3 119.442468) (end 112.432532 131.575) (width 0.25) (layer "F.Cu") (net 19))
-  (segment (start 100.3 103.8) (end 93.8 103.8) (width 0.25) (layer "F.Cu") (net 19))
-  (segment (start 112.432532 131.575) (end 128.700739 131.575) (width 0.25) (layer "F.Cu") (net 19))
+  (segment (start 140.400739 136.675) (end 133.800739 136.675) (width 0.25) (layer "F.Cu") (net 19))
+  (segment (start 99.975 102.625) (end 99.975 109.375) (width 0.25) (layer "F.Cu") (net 19))
+  (segment (start 101.3 101.3) (end 99.975 102.625) (width 0.25) (layer "F.Cu") (net 19))
+  (segment (start 149.440739 127.635) (end 140.400739 136.675) (width 0.25) (layer "F.Cu") (net 19))
+  (segment (start 99.975 109.375) (end 101.3 110.7) (width 0.25) (layer "F.Cu") (net 19))
+  (segment (start 101.3 110.7) (end 107.825739 110.7) (width 0.25) (layer "B.Cu") (net 19))
+  (segment (start 107.825739 110.7) (end 133.800739 136.675) (width 0.25) (layer "B.Cu") (net 19))
+  (segment (start 101.3 110.7) (end 94.8 110.7) (width 0.25) (layer "B.Cu") (net 19))
   (zone (net 1) (net_name "GND") (layer "B.Cu") (hatch edge 0.5)
     (connect_pads (clearance 0.508))
